File: Hardware/HighBitADCDAC/2656.brd (EAGLE design)
At the start: 65 x 56 mm, 34 parts, among them IC2 LM317, J1 SR_CONNECTOR_2X20, U1 LTC2656, U2 LTC2418, U5 SN74LS138D, U6 SN74HC595DR

Commit message: Add files via upload
Parts:
- moved J1 0.15 mm to (35.6, 59.8)
